Commit message: multi cam support

File: src/hiwonder_simulations/hiwonder_description/urdf/gazebo/arm.gazebo.xacro (robot description, xacro)
@@ -8,8 +8,11 @@
     </xacro:macro>
     <xacro:model_color link_name="link1"                color_name="black"/>
+    <xacro:model_color link_name="camera_connect_link"  color_name="black"/>
+    <xacro:model_color link_name="servo_link1"          color_name="black"/>
     <xacro:model_color link_name="link2"                color_name="black"/>
     <xacro:model_color link_name="link3"                color_name="black"/>
     <xacro:model_color link_name="link4"                color_name="black"/>
-    <xacro:model_color link_name="link4"                color_name="black"/>
-    <xacro:model_color link_name="gripper_base"         color_name="black"/>
+    <xacro:model_color link_name="link5"                color_name="black"/>
+    <xacro:model_color link_name="servo_link2"          color_name="black"/>
+    <xacro:model_color link_name="gripper_link"         color_name="black"/>
 </robot>

File: src/hiwonder_simulations/hiwonder_description/urdf/gazebo/arm.transmission.xacro (robot description, xacro)
@@ -17,3 +17,4 @@
     <xacro:SimpleTransmissionPosition joint="joint3" />
     <xacro:SimpleTransmissionPosition joint="joint4" />
+    <xacro:SimpleTransmissionPosition joint="joint5" />
 </robot>

File: src/hiwonder_simulations/hiwonder_description/urdf/gazebo/depth_camera.gazebo.xacro (robot description, xacro)
@@ -8,4 +8,5 @@
         </gazebo>
     </xacro:macro>
-    <xacro:model_color link_name="depth_cam_link"    color_name="black"/>
+    <xacro:model_color link_name="depth_cam_link"       color_name="black"/>
+    <xacro:model_color link_name="depth_cam_link_arm"   color_name="black"/>
 </robot>

File: src/hiwonder_simulations/hiwonder_description/urdf/gazebo/gripper.gazebo.xacro (robot description, xacro)
@@ -5,11 +5,9 @@
             <joint>r_joint</joint>
             <mimicJoint>r_out_joint</mimicJoint>
-            <multiplier>-1</multiplier>
-            <offset>0.0</offset>
         </plugin>
         <plugin name="mimic_plugin_r_in_link" filename="libroboticsgroup_upatras_gazebo_mimic_joint_plugin.so">
             <joint>r_joint</joint>
             <mimicJoint>r_in_joint</mimicJoint>
-            <multiplier>1</multiplier>
+            <multiplier>-1</multiplier>
             <offset>0.0</offset>
         </plugin>

File: src/hiwonder_simulations/hiwonder_description/urdf/roslander.gazebo.xacro (robot description, xacro)
@@ -1,5 +1,5 @@
 <?xml version="1.0" encoding="utf-8"?>
 <robot name="hiwonder" xmlns:xacro="http://ros.org/wiki/xacro">
-    <xacro:property name="mono_type"      value="$(env MONO_TYPE)"/>
+    <xacro:property name="camera_type"      value="$(env DEPTH_CAMERA_TYPE)"/>
     <xacro:include filename="$(find hiwonder_description)/urdf/roslander.xacro"/>
     <xacro:include filename="$(find hiwonder_description)/urdf/gazebo/car.gazebo.xacro"/>
@@ -7,10 +7,9 @@
     <xacro:include filename="$(find hiwonder_description)/urdf/gazebo/depth_camera.gazebo.xacro"/>
     <xacro:include filename="$(find hiwonder_description)/urdf/gazebo/lidar.gazebo.xacro"/>
-    <xacro:if value="${mono_type != 'None'}">
+    <xacro:if value="${camera_type != 'AstraProPlus'}">
         <xacro:include filename="$(find hiwonder_description)/urdf/gazebo/arm.transmission.xacro"/>
         <xacro:include filename="$(find hiwonder_description)/urdf/gazebo/arm.gazebo.xacro"/>
         <xacro:include filename="$(find hiwonder_description)/urdf/gazebo/gripper.transmission.xacro"/>
         <xacro:include filename="$(find hiwonder_description)/urdf/gazebo/gripper.gazebo.xacro"/>
-        <xacro:include filename="$(find hiwonder_description)/urdf/gazebo/usb_camera.gazebo.xacro"/>
     </xacro:if>
 </robot>

File: src/hiwonder_simulations/hiwonder_description/urdf/roslander.urdf.xacro (robot description, xacro)
@@ -167,5 +167,5 @@
   </joint>
   <link
-    name="depth_cam_link">
+    name="astra_camera_link">
     <visual>
       <origin
@@ -180,5 +180,5 @@
   </link>
   <joint
-    name="depth_cam_joint"
+    name="astra_camera_joint"
     type="fixed">
     <origin
@@ -188,5 +188,5 @@
       link="screen_link" />
     <child
-      link="depth_cam_link" />
+      link="astra_camera_link" />
     <axis
       xyz="0 0 0" />
@@ -355,14 +355,15 @@
     <inertial>
       <origin
-        xyz="0.000117652200128613 0.00166481375778722 0.0168007196434552"
-        rpy="0 0 0" />
-      <mass value="0.00001" />
-      <inertia
-        ixx="10"
-        ixy="0"
-        ixz="0"
-        iyy="10"
-        iyz="0"
-        izz="10" />
+        xyz="-0.000261855576526311 0.000239368359066633 0.0220971301535388"
+        rpy="0 0 0" />
+      <mass
+        value="0.00959141779390409" />
+      <inertia
+        ixx="7.94977139591732E-06"
+        ixy="-8.29446018776969E-10"
+        ixz="5.6880898756802E-08"
+        iyy="4.29063067361656E-06"
+        iyz="-1.84622131688891E-10"
+        izz="5.33833388813501E-06" />
     </inertial>
     <visual>
@@ -390,5 +391,5 @@
     type="revolute">
     <origin
-      xyz="0 0 0.129360132190811"
+      xyz="0 0 0.129444631186569"
       rpy="0 0 0" />
     <parent
@@ -405,36 +406,139 @@
   </joint>
   <link
-    name="gripper_base">
-    <inertial>
-      <origin
-        xyz="0.0135164471754075 -0.00245409302071614 0.0255243476105937"
-        rpy="0 0 0" />
-      <mass
-        value="0.0187986809487493" />
-      <inertia
-        ixx="4.18626999238256E-06"
-        ixy="-2.76258595538016E-08"
-        ixz="-7.69570071724482E-09"
-        iyy="1.60184662496099E-06"
-        iyz="2.25420771711905E-08"
-        izz="3.29280750879291E-06" />
-    </inertial>
-    <visual>
-      <origin
-        xyz="0 0 0"
-        rpy="0 0 0" />
-      <geometry>
-        <mesh
-          filename="package://hiwonder_description/meshes/gripper_base.STL" />
-      </geometry>
-      <material name="black"/>
-    </visual>
-    <collision>
-      <origin
-        xyz="0 0 0"
-        rpy="0 0 0" />
-      <geometry>
-        <mesh
-          filename="package://hiwonder_description/meshes/gripper_base.STL" />
+    name="servo_link2">
+    <inertial>
+      <origin
+        xyz="0.00829457691057159 0.000114732113040695 -0.0125525321145837"
+        rpy="0 0 0" />
+      <mass
+        value="0.00701021225113507" />
+      <inertia
+        ixx="6.10646998888003E-07"
+        ixy="1.66839713815154E-09"
+        ixz="-2.07626862362467E-08"
+        iyy="9.477990166652E-07"
+        iyz="5.12927100881908E-09"
+        izz="1.44691449724265E-06" />
+    </inertial>
+    <visual>
+      <origin
+        xyz="0 0 0"
+        rpy="0 0 0" />
+      <geometry>
+        <mesh
+          filename="package://hiwonder_description/meshes/servo_link2.STL" />
+      </geometry>
+      <material name="black"/>
+    </visual>
+    <collision>
+      <origin
+        xyz="0 0 0"
+        rpy="0 0 0" />
+      <geometry>
+        <mesh
+          filename="package://hiwonder_description/meshes/servo_link2.STL" />
+      </geometry>
+    </collision>
+  </link>
+  <joint
+    name="servo_joint2"
+    type="fixed">
+    <origin
+      xyz="0 0 0.0544833339503674"
+      rpy="0 0 0" />
+    <parent
+      link="link4" />
+    <child
+      link="servo_link2" />
+    <axis
+      xyz="0 0 0" />
+  </joint>
+  <link
+    name="link5">
+    <inertial>
+      <origin
+        xyz="-5.40141895711381E-05 -8.30141354428709E-06 0.00351551092860852"
+        rpy="0 0 0" />
+      <mass
+        value="0.00101775298619909" />
+      <inertia
+        ixx="2.35834256739382E-08"
+        ixy="-1.92177809145012E-12"
+        ixz="-3.88572739181837E-12"
+        iyy="2.35740360938003E-08"
+        iyz="-1.1228386368903E-13"
+        izz="4.40224050991292E-08" />
+    </inertial>
+    <visual>
+      <origin
+        xyz="0 0 0"
+        rpy="0 0 0" />
+      <geometry>
+        <mesh
+          filename="package://hiwonder_description/meshes/link5.STL" />
+      </geometry>
+      <material name="black"/>
+    </visual>
+    <collision>
+      <origin
+        xyz="0 0 0"
+        rpy="0 0 0" />
+      <geometry>
+        <mesh
+          filename="package://hiwonder_description/meshes/link5.STL" />
+      </geometry>
+    </collision>
+  </link>
+  <joint
+    name="joint5"
+    type="revolute">
+    <origin
+      xyz="0 0 0"
+      rpy="0 0 0" />
+    <parent
+      link="servo_link2" />
+    <child
+      link="link5" />
+    <axis
+      xyz="0 0 -1" />
+    <limit
+      lower="-2.09"
+      upper="2.09"
+      effort="1000"
+      velocity="10" />
+  </joint>
+  <link
+    name="gripper_link">
+    <inertial>
+      <origin
+        xyz="0.0145481835889059 -0.00315257290321308 0.0253492053712461"
+        rpy="0 0 0" />
+      <mass
+        value="0.0174988490314194" />
+      <inertia
+        ixx="4.12615692688456E-06"
+        ixy="-2.75102939068049E-08"
+        ixz="-7.61180742281118E-09"
+        iyy="1.57023365316943E-06"
+        iyz="2.2563082379695E-08"
+        izz="3.2612101868791E-06" />
+    </inertial>
+    <visual>
+      <origin
+        xyz="0 0 0"
+        rpy="0 0 0" />
+      <geometry>
+        <mesh
+          filename="package://hiwonder_description/meshes/gripper_link.STL" />
+      </geometry>
+      <material name="black"/>
+    </visual>
+    <collision>
+      <origin
+        xyz="0 0 0"
+        rpy="0 0 0" />
+      <geometry>
+        <mesh
+          filename="package://hiwonder_description/meshes/gripper_link.STL" />
       </geometry>
     </collision>
@@ -444,12 +548,19 @@
     type="fixed">
     <origin
-      xyz="0 0 0.0415523547092036"
-      rpy="0 0 0" />
-    <parent
-      link="link4" />
-    <child
-      link="gripper_base" />
-    <axis
-      xyz="0 0 0" />
+      xyz="0 0 0.0054388"
+      rpy="0 0 0" />
+    <parent
+      link="link5" />
+    <child
+      link="gripper_link" />
+    <axis
+      xyz="0 0 0" />
+  </joint>
+  <!-- end effector link -->
+  <link name="end_effector_link" />
+  <joint name="end_effector_joint" type="fixed">
+    <origin xyz="0 0 0.08" rpy="0 0 0"/>
+    <parent link="link5"/>
+    <child link="end_effector_link"/>
   </joint>
   <link
@@ -457,15 +568,15 @@
     <inertial>
       <origin
-        xyz="4.5917753844606E-05 0.000541568299117931 0.00625139747060544"
-        rpy="0 0 0" />
-      <mass
-        value="0.00206273118071422" />
-      <inertia
-        ixx="3.97236083071195E-07"
-        ixy="-2.70823664638678E-10"
-        ixz="-2.16820413734473E-09"
-        iyy="3.22499205032185E-07"
-        iyz="1.07452392164753E-08"
-        izz="7.78636035301087E-08" />
+        xyz="0.00154652142582958 0.000534112070478834 0.00624030428121536"
+        rpy="0 0 0" />
+      <mass
+        value="0.00206265647704866" />
+      <inertia
+        ixx="3.97215843669342E-07"
+        ixy="-2.75699120579387E-10"
+        ixz="-2.19901048536124E-09"
+        iyy="3.22472627342115E-07"
+        iyz="1.07303783544668E-08"
+        izz="7.78708186672131E-08" />
     </inertial>
     <visual>
@@ -493,17 +604,17 @@
     type="revolute">
     <origin
-      xyz="-0.0056586 -0.012538 0.027102"
-      rpy="0 0 0" />
-    <parent
-      link="gripper_base" />
+      xyz="-0.0073166 -0.013992 0.027059"
+      rpy="0 0 0" />
+    <parent
+      link="gripper_link" />
     <child
       link="r_link" />
     <axis
-      xyz="-1 0 0" />
+      xyz="0.99996 -0.004699 -0.0070434" />
     <limit
       lower="-1.57"
       upper="1.57"
       effort="1000"
-      velocity="2" />
+      velocity="10" />
   </joint>
   <link
@@ -511,15 +622,15 @@
     <inertial>
       <origin
-        xyz="3.79169240065586E-05 -0.000411330229694192 0.00580564378864612"
-        rpy="0 0 0" />
-      <mass
-        value="0.00218935442813927" />
-      <inertia
-        ixx="4.05423576726065E-07"
-        ixy="3.5639084027101E-10"
-        ixz="-1.96705902005403E-09"
-        iyy="3.31275196418489E-07"
-        iyz="-8.75686731441383E-09"
-        izz="7.74603139284005E-08" />
+        xyz="0.0015384031888858 -0.000403232726847674 0.00579759783012201"
+        rpy="0 0 0" />
+      <mass
+        value="0.00218924933187322" />
+      <inertia
+        ixx="4.0534152698165E-07"
+        ixy="3.60077827494503E-10"
+        ixz="-1.99675888093364E-09"
+        iyy="3.31222174181852E-07"
+        iyz="-8.79337758250917E-09"
+        izz="7.74319582642917E-08" />
     </inertial>
     <visual>
@@ -547,17 +658,17 @@
     type="revolute">
     <origin
-      xyz="-0.0056772 0.015434 0.027105"
-      rpy="0 0 0" />
-    <parent
-      link="gripper_base" />
+      xyz="-0.0073352 0.013977 0.027057"
+      rpy="0 0 0" />
+    <parent
+      link="gripper_link" />
     <child
       link="l_link" />
     <axis
-      xyz="-1 0 0" />
+      xyz="0.99997 0.0055811 -0.0058397" />
     <limit
       lower="-1.57"
       upper="1.57"
       effort="1000"
-      velocity="2" />
+      velocity="10" />
     <mimic
       joint="r_joint"
@@ -566,56 +677,114 @@
   </joint>
   <link
-    name="r_in_link">
-    <inertial>
-      <origin
-        xyz="0.00460054659575418 -2.07965839691421E-05 0.0144687504641022"
-        rpy="0 0 0" />
-      <mass
-        value="0.000776937620409709" />
-      <inertia
-        ixx="9.8752111566072E-08"
-        ixy="-5.02144302953861E-12"
-        ixz="-6.7016858192728E-10"
-        iyy="9.76692470887995E-08"
-        iyz="-2.41388732380185E-13"
-        izz="2.25760020432699E-09" />
-    </inertial>
-    <visual>
-      <origin
-        xyz="0 0 0"
-        rpy="0 0 0" />
-      <geometry>
-        <mesh
-          filename="package://hiwonder_description/meshes/r_in_link.STL" />
-      </geometry>
-      <material name="black"/>
-    </visual>
-    <collision>
-      <origin
-        xyz="0 0 0"
-        rpy="0 0 0" />
-      <geometry>
-        <mesh
-          filename="package://hiwonder_description/meshes/r_in_link.STL" />
-      </geometry>
-    </collision>
-  </link>
-  <joint
-    name="r_in_joint"
+    name="l_in_link">
+    <inertial>
+      <origin
+        xyz="0.00610191812065245 2.91459132896708E-05 0.0144573768632076"
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
File: src/hiwonder_simulations/hiwonder_description/urdf/roslander.xacro (robot description, xacro)
@@ -1,9 +1,9 @@
 <?xml version="1.0" encoding="utf-8"?>
 <robot name="hiwonder" xmlns:xacro="http://ros.org/wiki/xacro">
-    <xacro:property name="mono_type"      value="$(env MONO_TYPE)"/>
-    <xacro:if value="${mono_type == 'None'}">
+    <xacro:property name="camera_type"      value="$(env DEPTH_CAMERA_TYPE)"/>
+    <xacro:if value="${camera_type == 'AstraProPlus'}">
         <xacro:include filename="$(find hiwonder_description)/urdf/roslander_without_arm.urdf.xacro"/>
     </xacro:if>
-    <xacro:if value="${mono_type != 'None'}">
+    <xacro:if value="${camera_type != 'AstraProPlus'}">
         <xacro:include filename="$(find hiwonder_description)/urdf/roslander.urdf.xacro"/>
     </xacro:if>
