Commit message: fix sim

File: src/hiwonder_simulations/hiwonder_description/urdf/gazebo/imu.gazebo.xacro (robot description, xacro)
@@ -5,6 +5,6 @@
       <alwaysOn>true</alwaysOn>
       <bodyName>imu_link</bodyName>
-      <frameName>imu_link</frameName>
-      <topicName>imu_data</topicName>
+      <frameName>imu_frame</frameName>
+      <topicName>imu</topicName>
       <serviceName>imu_service</serviceName>
       <gaussianNoise>0.0</gaussianNoise>

File: src/hiwonder_simulations/hiwonder_description/urdf/gazebo/lidar.gazebo.xacro (robot description, xacro)
@@ -1,5 +1,5 @@
 <?xml version="1.0" encoding="utf-8" ?>
 <robot xmlns:xacro="http://ros.org/wiki/xacro">
-    <gazebo reference="lidar_frame">
+    <gazebo reference="lidar_sim_frame">
       <sensor type="ray" name="lidar">
         <pose>0 0 0 0 0 0</pose>
@@ -28,5 +28,5 @@
         <plugin name="gazebo_rplidar" filename="libgazebo_ros_laser.so">
           <topicName>scan_raw</topicName>
-          <frameName>lidar_frame</frameName>
+          <frameName>$(arg lidar_frame)</frameName>
         </plugin>
       </sensor>

File: src/hiwonder_simulations/hiwonder_description/urdf/roslander.gazebo.xacro (robot description, xacro)
@@ -7,4 +7,5 @@
     <xacro:include filename="$(find hiwonder_description)/urdf/gazebo/depth_camera.gazebo.xacro"/>
     <xacro:include filename="$(find hiwonder_description)/urdf/gazebo/lidar.gazebo.xacro"/>
+    <xacro:include filename="$(find hiwonder_description)/urdf/gazebo/imu.gazebo.xacro"/>
     <xacro:if value="${camera_type != 'AstraProPlus'}">
         <xacro:include filename="$(find hiwonder_description)/urdf/gazebo/arm.transmission.xacro"/>

File: src/hiwonder_simulations/hiwonder_description/urdf/roslander.urdf.xacro (robot description, xacro)
@@ -1168,4 +1168,12 @@
       xyz="0 0 0" />
   </joint>
+  <link name="lidar_sim_frame" />
+  <joint
+    name="lidar_sim_frame_joint"
+    type="fixed">
+    <origin xyz="0 0 0" rpy="0 0 ${M_PI}" />
+    <parent link="lidar_link" />
+    <child link="lidar_sim_frame" />
+  </joint>
   <xacro:if value="${lidar in ['A1', 'A2', 'S2L']}">
     <xacro:include filename="$(find hiwonder_description)/urdf/lidar_a1.urdf.xacro"/>
