Commit message: clean

File: src/hiwonder_simulations/hiwonder_description/urdf/inertial_matrix.xacro (robot description, xacro)
@@ -1,4 +1,4 @@
 <?xml version="1.0" encoding="utf-8"?>
-<robot name="inertial_matrix" xmlns:xacro="http://ros.org/wiki/xacro">
+<robot name="hiwonder" xmlns:xacro="http://ros.org/wiki/xacro">
   <xacro:property name="M_PI" value="3.1415926535897931" />
   <!-- Macro for inertia matrix -->
@@ -27,9 +27,6 @@
     </inertial>
   </xacro:macro>
-  <xacro:macro name="box_inertial" params="m w h d x y z">
-      <inertial>
-      <origin
-        xyz="${x} ${y} ${z}"
-        rpy="0 0 0" />
+  <xacro:macro name="box_inertial" params="m w h d">
+    <inertial>
       <mass value="${m}" />
       <inertia

File: src/hiwonder_simulations/hiwonder_description/urdf/lidar_a1.urdf.xacro (robot description, xacro)
@@ -1,10 +1,9 @@
 <?xml version="1.0" encoding="utf-8"?>
 <robot name="lidar_a1" xmlns:xacro="http://ros.org/wiki/xacro" >
-  <xacro:property name="M_PI" value="3.1415926535897931"/>
   <link name="lidar_frame" />
   <joint
     name="lidar_frame_joint"
     type="fixed">
-    <origin xyz="0 0 0" rpy="0 0 ${M_PI}" />
+    <origin xyz="0 0 0" rpy="0 0 0" />
     <parent link="lidar_link" />
     <child link="lidar_frame" />

File: src/hiwonder_simulations/hiwonder_description/urdf/lidar_g4.urdf.xacro (robot description, xacro)
@@ -1,4 +1,4 @@
 <?xml version="1.0" encoding="utf-8"?>
-<robot name="lidar_g4" xmlns:xacro="http://ros.org/wiki/xacro" >
+<robot name="lidar_a1" xmlns:xacro="http://ros.org/wiki/xacro" >
   <xacro:property name="M_PI" value="3.1415926535897931"/>
   <link name="lidar_frame" />
@@ -6,5 +6,5 @@
     name="lidar_frame_joint"
     type="fixed">
-    <origin xyz="0 0 0" rpy="0 0 0" />
+    <origin xyz="0 0 0" rpy="0 0 ${M_PI}" />
     <parent link="lidar_link" />
     <child link="lidar_frame" />

File: src/hiwonder_simulations/hiwonder_description/urdf/materials.xacro (robot description, xacro)
@@ -1,4 +1,4 @@
 <?xml version="1.0"?>
-<robot name="material" xmlns:xacro="http://ros.org/wiki/xacro">
+<robot>
     <material name="black">
         <color rgba="0.1 0.1 0.1 1.0"/>
